File: Hardware/Kicad/PureAir/PureAir.kicad_sch (KiCad schematic)
At the start: 8 parts, among them SW1 SW_Push, U1 DHT22, U2 MQ-2

Commit message: Start Creating footPrint
Parts:
- U1: footprint (none) -> LibrarPureAirLib:Dht22
- U2: footprint (none) -> LibrarPureAirLib:Mq2-Sens
Changed lines of the file:
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@@
     (property "Reference" "U1" (id 0) (at 90.17 109.22 0))
     (property "Value" "DHT22" (id 1) (at 90.17 111.76 0))
-    (property "Footprint" "" (id 2) (at 90.17 119.38 0)
+    (property "Footprint" "LibrarPureAirLib:Dht22" (id 2) (at 90.17 119.38 0)
       (effects (font (size 1.27 1.27)) hide)
     )
@@
       (effects (font (size 1.27 1.27)) (justify left))
     )
-    (property "Footprint" "" (id 2) (at 160.02 111.76 0)
+    (property "Footprint" "LibrarPureAirLib:Mq2-Sens" (id 2) (at 160.02 111.76 0)
       (effects (font (size 1.27 1.27)) hide)
     )
@@
     )
     (path "/143bba8f-2ae4-4e97-b9f1-5ac6e9301742"
-      (reference "U1") (unit 1) (value "DHT22") (footprint "")
+      (reference "U1") (unit 1) (value "DHT22") (footprint "LibrarPureAirLib:Dht22")
     )
     (path "/15ffa9e7-a1d0-42e0-a0d1-fd47941e5abb"
-      (reference "U2") (unit 1) (value "MQ-2") (footprint "")
-    )
-  )
+      (reference "U2") (unit 1) (value "MQ-2") (footprint "LibrarPureAirLib:Mq2-Sens")
+    )
+  )
